Commit message: Add ability to override default initial position by passing a yaml file

File: panda_moveit_config/config/panda.ros2_control.xacro (robot description, xacro)
@@ -1,5 +1,17 @@
 <?xml version="1.0"?>
 <robot xmlns:xacro="http://www.ros.org/wiki/xacro">
-    <xacro:macro name="panda_ros2_control" params="name">
+    <xacro:macro name="panda_ros2_control" params="name initial_positions_file">
+        <xacro:if value="${initial_positions_file == ''}">
+            <xacro:property name="initial_positions" value="${dict(panda_joint1=0.0,
+                                                                   panda_joint2=-0.785,
+                                                                   panda_joint3=0.0,
+                                                                   panda_joint4=-2.356,
+                                                                   panda_joint5=0.0,
+                                                                   panda_joint6=1.571,
+                                                                   panda_joint7=0.785)}"/>
+        </xacro:if>
+        <xacro:unless value="${initial_positions_file == ''}">
+            <xacro:property name="initial_positions" value="${load_yaml(initial_positions_file)['initial_positions']}"/>
+        </xacro:unless>
         <ros2_control name="${name}" type="system">
             <hardware>
@@ -7,5 +19,5 @@
             </hardware>
             <joint name="panda_joint1">
-                <param name="initial_position">0.0</param>
+                <param name="initial_position">${initial_positions['panda_joint1']}</param>
                 <command_interface name="position" />
                 <state_interface name="position"/>
@@ -13,5 +25,5 @@
             </joint>
             <joint name="panda_joint2">
-                <param name="initial_position">-0.785</param>
+                <param name="initial_position">${initial_positions['panda_joint2']}</param>
                 <command_interface name="position" />
                 <state_interface name="position"/>
@@ -19,5 +31,5 @@
             </joint>
             <joint name="panda_joint3">
-                <param name="initial_position">0.0</param>
+                <param name="initial_position">${initial_positions['panda_joint3']}</param>
                 <command_interface name="position" />
                 <state_interface name="position"/>
@@ -25,5 +37,5 @@
             </joint>
             <joint name="panda_joint4">
-                <param name="initial_position">-2.356</param>
+                <param name="initial_position">${initial_positions['panda_joint4']}</param>
                 <command_interface name="position" />
                 <state_interface name="position"/>
@@ -31,5 +43,5 @@
             </joint>
             <joint name="panda_joint5">
-                <param name="initial_position">0.0</param>
+                <param name="initial_position">${initial_positions['panda_joint5']}</param>
                 <command_interface name="position" />
                 <state_interface name="position"/>
@@ -37,5 +49,5 @@
             </joint>
             <joint name="panda_joint6">
-                <param name="initial_position">1.571</param>
+                <param name="initial_position">${initial_positions['panda_joint6']}</param>
                 <command_interface name="position" />
                 <state_interface name="position"/>
@@ -43,5 +55,5 @@
             </joint>
             <joint name="panda_joint7">
-                <param name="initial_position">0.785</param>
+                <param name="initial_position">${initial_positions['panda_joint7']}</param>
                 <command_interface name="position" />
                 <state_interface name="position"/>

File: panda_moveit_config/config/panda.urdf.xacro (robot description, xacro)
@@ -1,8 +1,9 @@
 <?xml version="1.0"?>
 <robot xmlns:xacro="http://www.ros.org/wiki/xacro" name="panda">
+    <xacro:arg name="initial_positions_file" default="" />
     <!-- Import panda urdf file -->
     <xacro:include filename="$(find moveit_resources_panda_description)/urdf/panda.urdf" />
     <!-- Import panda ros2_control description -->
     <xacro:include filename="panda.ros2_control.xacro" />
-    <xacro:panda_ros2_control name="PandaFakeSystem" />
+    <xacro:panda_ros2_control name="PandaFakeSystem" initial_positions_file="$(arg initial_positions_file)"/>
 </robot>

Commit message: No initial velocity conditions

File: panda_moveit_config/config/panda.ros2_control.xacro (robot description, xacro)
@@ -3,5 +3,4 @@
     <xacro:macro name="panda_ros2_control" params="name initial_positions_file">
         <xacro:property name="initial_positions" value="${load_yaml(initial_positions_file)['initial_positions']}"/>
-        <xacro:property name="initial_velocities" value="${load_yaml(initial_positions_file)['initial_velocities']}"/>
         <ros2_control name="${name}" type="system">
             <hardware>
@@ -13,7 +12,5 @@
                   <param name="initial_value">${initial_positions['panda_joint1']}</param>
                 </state_interface>
-                <state_interface name="velocity">
-                  <param name="initial_value">${initial_velocities['panda_joint1']}</param>
-                </state_interface>
+                <state_interface name="velocity"/>
             </joint>
             <joint name="panda_joint2">
@@ -22,7 +19,5 @@
                   <param name="initial_value">${initial_positions['panda_joint2']}</param>
                 </state_interface>
-                <state_interface name="velocity">
-                  <param name="initial_value">${initial_velocities['panda_joint2']}</param>
-                </state_interface>
+                <state_interface name="velocity"/>
             </joint>
             <joint name="panda_joint3">
@@ -31,7 +26,5 @@
                   <param name="initial_value">${initial_positions['panda_joint3']}</param>
                 </state_interface>
-                <state_interface name="velocity">
-                  <param name="initial_value">${initial_velocities['panda_joint3']}</param>
-                </state_interface>
+                <state_interface name="velocity"/>
             </joint>
             <joint name="panda_joint4">
@@ -40,7 +33,5 @@
                   <param name="initial_value">${initial_positions['panda_joint4']}</param>
                 </state_interface>
-                <state_interface name="velocity">
-                  <param name="initial_value">${initial_velocities['panda_joint4']}</param>
-                </state_interface>
+                <state_interface name="velocity"/>
             </joint>
             <joint name="panda_joint5">
@@ -49,7 +40,5 @@
                   <param name="initial_value">${initial_positions['panda_joint5']}</param>
                 </state_interface>
-                <state_interface name="velocity">
-                  <param name="initial_value">${initial_velocities['panda_joint5']}</param>
-                </state_interface>
+                <state_interface name="velocity"/>
             </joint>
             <joint name="panda_joint6">
@@ -58,7 +47,5 @@
                   <param name="initial_value">${initial_positions['panda_joint6']}</param>
                 </state_interface>
-                <state_interface name="velocity">
-                  <param name="initial_value">${initial_velocities['panda_joint6']}</param>
-                </state_interface>
+                <state_interface name="velocity"/>
             </joint>
             <joint name="panda_joint7">
@@ -67,7 +54,5 @@
                   <param name="initial_value">${initial_positions['panda_joint7']}</param>
                 </state_interface>
-                <state_interface name="velocity">
-                  <param name="initial_value">${initial_velocities['panda_joint7']}</param>
-                </state_interface>
+                <state_interface name="velocity"/>
             </joint>
         </ros2_control>

File: panda_moveit_config/config/panda_hand.ros2_control.xacro (robot description, xacro)
@@ -11,7 +11,5 @@
                   <param name="initial_value">0.0</param>
                 </state_interface>
-                <state_interface name="velocity">
-                  <param name="initial_value">0.0</param>
-                </state_interface>
+                <state_interface name="velocity"/>
             </joint>
             <joint name="panda_finger_joint2">
@@ -22,7 +20,5 @@
                   <param name="initial_value">0.0</param>
                 </state_interface>
-                <state_interface name="velocity">
-                  <param name="initial_value">0.0</param>
-                </state_interface>
+                <state_interface name="velocity"/>
             </joint>
         </ros2_control>

Commit message: Removed warning about using deprecated load_yaml method. Now using xacro.load_yaml.

File: panda_moveit_config/config/panda.ros2_control.xacro (robot description, xacro)
@@ -2,5 +2,5 @@
 <robot xmlns:xacro="http://www.ros.org/wiki/xacro">
     <xacro:macro name="panda_ros2_control" params="name initial_positions_file">
-        <xacro:property name="initial_positions" value="${load_yaml(initial_positions_file)['initial_positions']}"/>
+        <xacro:property name="initial_positions" value="${xacro.load_yaml(initial_positions_file)['initial_positions']}"/>
         <ros2_control name="${name}" type="system">
             <hardware>

Commit message: Add xacro parameter to select ros2_control hardware interface type

File: panda_moveit_config/config/panda.ros2_control.xacro (robot description, xacro)
@@ -1,9 +1,16 @@
 <?xml version="1.0"?>
 <robot xmlns:xacro="http://www.ros.org/wiki/xacro">
-    <xacro:macro name="panda_ros2_control" params="name initial_positions_file">
+    <xacro:macro name="panda_ros2_control" params="name initial_positions_file ros2_control_hardware_type">
         <xacro:property name="initial_positions" value="${xacro.load_yaml(initial_positions_file)['initial_positions']}"/>
         <ros2_control name="${name}" type="system">
             <hardware>
-                <plugin>mock_components/GenericSystem</plugin>
+                <xacro:if value="${ros2_control_hardware_type == 'mock_components'}">
+                    <plugin>mock_components/GenericSystem</plugin>
+                </xacro:if>
+                <xacro:if value="${ros2_control_hardware_type == 'isaac'}">
+                    <plugin>isaac_ros2_control/IsaacSystem</plugin>
+                    <param name="joint_commands_topic">/isaac_joint_commands</param>
+                    <param name="joint_states_topic">/isaac_joint_states</param>
+                </xacro:if>
             </hardware>
             <joint name="panda_joint1">

File: panda_moveit_config/config/panda_hand.ros2_control.xacro (robot description, xacro)
@@ -1,8 +1,15 @@
 <?xml version="1.0"?>
 <robot xmlns:xacro="http://www.ros.org/wiki/xacro">
-    <xacro:macro name="panda_hand_ros2_control" params="name">
+    <xacro:macro name="panda_hand_ros2_control" params="name ros2_control_hardware_type">
         <ros2_control name="${name}" type="system">
             <hardware>
-                <plugin>mock_components/GenericSystem</plugin>
+                <xacro:if value="${ros2_control_hardware_type == 'mock_components'}">
+                    <plugin>mock_components/GenericSystem</plugin>
+                </xacro:if>
+                <xacro:if value="${ros2_control_hardware_type == 'isaac'}">
+                    <plugin>isaac_ros2_control/IsaacSystem</plugin>
+                    <param name="joint_commands_topic">/isaac_joint_commands</param>
+                    <param name="joint_states_topic">/isaac_joint_states</param>
+                </xacro:if>
             </hardware>
             <joint name="panda_finger_joint1">

Commit message: Replace Isaac with TopicBased (#163)

File: panda_moveit_config/config/panda.ros2_control.xacro (robot description, xacro)
@@ -1,9 +1,16 @@
 <?xml version="1.0"?>
 <robot xmlns:xacro="http://www.ros.org/wiki/xacro">
-    <xacro:macro name="panda_ros2_control" params="name initial_positions_file">
+    <xacro:macro name="panda_ros2_control" params="name initial_positions_file ros2_control_hardware_type">
         <xacro:property name="initial_positions" value="${xacro.load_yaml(initial_positions_file)['initial_positions']}"/>
         <ros2_control name="${name}" type="system">
             <hardware>
-                <plugin>mock_components/GenericSystem</plugin>
+                <xacro:if value="${ros2_control_hardware_type == 'mock_components'}">
+                    <plugin>mock_components/GenericSystem</plugin>
+                </xacro:if>
+                <xacro:if value="${ros2_control_hardware_type == 'isaac'}">
+                    <plugin>topic_based_ros2_control/TopicBasedSystem</plugin>
+                    <param name="joint_commands_topic">/isaac_joint_commands</param>
+                    <param name="joint_states_topic">/isaac_joint_states</param>
+                </xacro:if>
             </hardware>
             <joint name="panda_joint1">

Commit message: Add xacro option for Ignition support

File: panda_moveit_config/config/panda.ros2_control.xacro (robot description, xacro)
@@ -7,4 +7,7 @@
                 <xacro:if value="${ros2_control_hardware_type == 'mock_components'}">
                     <plugin>mock_components/GenericSystem</plugin>
+                </xacro:if>
+                <xacro:if value="${ros2_control_hardware_type == 'sim_ignition'}">
+                    <plugin>ign_ros2_control/IgnitionSystem</plugin>
                 </xacro:if>
                 <xacro:if value="${ros2_control_hardware_type == 'isaac'}">
@@ -64,4 +67,17 @@
             </joint>
         </ros2_control>
+        <xacro:if value="${ros2_control_hardware_type == 'sim_ignition'}">
+          <link name="world"/>
+          <joint name="panda_world" type="fixed">
+              <origin rpy="0 0 0" xyz="0 0 0.0" />
+              <parent link="world" />
+              <child link="panda_link0" />
+          </joint>
+          <gazebo>
+            <plugin filename="libign_ros2_control-system.so" name="ign_ros2_control::IgnitionROS2ControlPlugin">
+              <parameters>$(find moveit_resources_panda_moveit_config)/config/ros2_controllers.yaml</parameters>
+            </plugin>
+          </gazebo>
+        </xacro:if>
     </xacro:macro>
 </robot>

File: panda_moveit_config/config/panda_hand.ros2_control.xacro (robot description, xacro)
@@ -6,4 +6,7 @@
                 <xacro:if value="${ros2_control_hardware_type == 'mock_components'}">
                     <plugin>mock_components/GenericSystem</plugin>
+                </xacro:if>
+                <xacro:if value="${ros2_control_hardware_type == 'sim_ignition'}">
+                    <plugin>ign_ros2_control/IgnitionSystem</plugin>
                 </xacro:if>
                 <xacro:if value="${ros2_control_hardware_type == 'isaac'}">
