Commit message: Apply inertial,dynamics and fix mesh locations

File: panda_description/urdf/panda.urdf (robot description, URDF)
Before this commit: robot panda, 12 links, 11 joints
Links:
- link panda_hand: mass None -> 0.73; geometry collision mesh filename=file://$(find moveit_resources_panda_description)/meshes/co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; visual mesh filename=file://$(find moveit_resources_panda_description)/meshes/vi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
- link panda_leftfinger: mass None -> 0.015; geometry collision mesh filename=file://$(find moveit_resources_panda_description)/meshes/co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; visual mesh filename=file://$(find moveit_resources_panda_description)/meshes/vi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
- link panda_link0: mass None -> 0.629769; geometry collision mesh filename=file://$(find moveit_resources_panda_description)/meshes/co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; visual mesh filename=file://$(find moveit_resources_panda_description)/meshes/vi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
- link panda_link1: mass None -> 4.970684; geometry collision mesh filename=file://$(find moveit_resources_panda_description)/meshes/co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; visual mesh filename=file://$(find moveit_resources_panda_description)/meshes/vi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
- link panda_link2: mass None -> 0.646926; geometry collision mesh filename=file://$(find moveit_resources_panda_description)/meshes/co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; visual mesh filename=file://$(find moveit_resources_panda_description)/meshes/vi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
- link panda_link3: mass None -> 3.228604; geometry collision mesh filename=file://$(find moveit_resources_panda_description)/meshes/co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; visual mesh filename=file://$(find moveit_resources_panda_description)/meshes/vi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
- link panda_link4: mass None -> 3.587895; geometry collision mesh filename=file://$(find moveit_resources_panda_description)/meshes/co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; visual mesh filename=file://$(find moveit_resources_panda_description)/meshes/vi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
- link panda_link5: mass None -> 1.225946; geometry collision mesh filename=file://$(find moveit_resources_panda_description)/meshes/co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; visual mesh filename=file://$(find moveit_resources_panda_description)/meshes/vi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
- link panda_link6: mass None -> 1.666555; geometry collision mesh filename=file://$(find moveit_resources_panda_description)/meshes/co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; visual mesh filename=file://$(find moveit_resources_panda_description)/meshes/vi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
- link panda_link7: mass None -> 7.35522E-1; geometry collision mesh filename=file://$(find moveit_resources_panda_description)/meshes/co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; visual mesh filename=file://$(find moveit_resources_panda_description)/meshes/vi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
- link panda_rightfinger: mass None -> 0.15; geometry collision mesh filename=file://$(find moveit_resources_panda_description)/meshes/co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; visual mesh filename=file://$(find moveit_resources_panda_description)/meshes/vi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
