Commit message: feat: Added gz as hardware type using ign_ros2_control

File: panda_description/urdf/panda.urdf.xacro (robot description, xacro)
@@ -5,4 +5,9 @@
 <!-- =================================================================================== -->
 <robot name="panda" xmlns:xacro="http://www.ros.org/wiki/xacro">
+    <link name="world"/>
+    <joint name="world_fixed" type="fixed">
+        <parent link="world"/>
+        <child link="panda_link0"/>
+    </joint>
     <link name="panda_link0">
         <visual>

File: panda_moveit_config/config/panda.ros2_control.xacro (robot description, xacro)
@@ -12,4 +12,7 @@
                     <param name="joint_commands_topic">/isaac_joint_commands</param>
                     <param name="joint_states_topic">/isaac_joint_states</param>
+                </xacro:if>
+                <xacro:if value="${ros2_control_hardware_type == 'gz'}">
+                    <plugin>gz_ros2_control/GazeboSimSystem</plugin>
                 </xacro:if>
             </hardware>

File: panda_moveit_config/config/panda.urdf.xacro (robot description, xacro)
@@ -2,5 +2,14 @@
 <robot xmlns:xacro="http://www.ros.org/wiki/xacro" name="panda">
     <xacro:arg name="initial_positions_file" default="initial_positions.yaml" />
-    <xacro:arg name="ros2_control_hardware_type" default="mock_components" />
+    <xacro:arg name="ros2_control_hardware_type" default="gz"/>
+    <xacro:property name="ros2_control_hardware_type_property" value="$(arg ros2_control_hardware_type)" />
+    <xacro:property name="initial_positions" value="${xacro.load_yaml(initial_positions_file)['initial_positions']}"/>
+    <xacro:if value="${ros2_control_hardware_type_property == 'gz'}">
+        <gazebo>
+            <plugin name="ign_ros2_control::IgnitionROS2ControlPlugin" filename="libign_ros2_control-system.so">
+                <parameters>$(find moveit_resources_panda_moveit_config)/config/ros2_controllers.yaml</parameters>
+            </plugin>
+        </gazebo>
+    </xacro:if>
     <!-- Import panda urdf file -->
     <xacro:include filename="$(find moveit_resources_panda_description)/urdf/panda.urdf.xacro" />

File: panda_moveit_config/config/panda_hand.ros2_control.xacro (robot description, xacro)
@@ -11,4 +11,7 @@
                     <param name="joint_commands_topic">/isaac_joint_commands</param>
                     <param name="joint_states_topic">/isaac_joint_states</param>
+                </xacro:if>
+                <xacro:if value="${ros2_control_hardware_type == 'gz'}">
+                    <plugin>gz_ros2_control/GazeboSimSystem</plugin>
                 </xacro:if>
             </hardware>
